File: hardware/BREAD_Slice_connProto.kicad_pcb (KiCad board)
At the start: 2 copper layers, 70 x 100 mm, 15 parts, among them J1 Conn_01x10_Female

Commit message: initial commit breaking off from Slice_TEMP
Parts:
- added J2: Conn_01x08, TerminalBlock_4Ucon:TerminalBlock_4Ucon_1x08_P3.50mm_Horizontal, F.Cu at (187.2, 83.2)
- added J3: Conn_01x08, TerminalBlock_4Ucon:TerminalBlock_4Ucon_1x08_P3.50mm_Horizontal, F.Cu at (187.1, 117.4)
Routing:
- net /D12: track 0.00 -> 82.5 mm
- net /D11: track 0.00 -> 81.8 mm
- net /D10: track 0.00 -> 81.3 mm
- net /D9: track 0.00 -> 80.8 mm
- net /D8: track 0.00 -> 80.3 mm
- net /D7: track 0.00 -> 79.8 mm
- net /D6: track 0.00 -> 79.3 mm
- net /D13: track 0.00 -> 75.5 mm
- net /A3: track 0.00 -> 35.2 mm
- net /A2: track 0.00 -> 34.8 mm
- net /A1: track 0.00 -> 34.4 mm
- net /A0: track 0.00 -> 34.0 mm
- net /A7: track 0.00 -> 33.9 mm
- net /AREF: track 0.00 -> 33.6 mm
- net /A6: track 0.00 -> 33.5 mm
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Other:
- board text added: "BREAD Slice Template: -> Conn SLC_TEMP R2 04-2025"
- board text removed: "BREAD Slice Template SLC_TEMP R3 04-2025"

Commit message: generated outputs to order
Parts:
- added J4: Conn_02x10_Odd_Even, Connector_PinHeader_2.54mm:PinHeader_2x10_P2.54mm_Vertical, F.Cu at (135.9, 59.1)
- added J5: Conn_02x10_Odd_Even, Connector_PinHeader_2.54mm:PinHeader_2x10_P2.54mm_Vertical, F.Cu at (149.2, 59.1)
- added J6: Conn_02x10_Odd_Even, Connector_PinHeader_2.54mm:PinHeader_2x10_P2.54mm_Vertical, F.Cu at (155.6, 59.1)
- added J7: Conn_02x10_Odd_Even, Connector_PinHeader_2.54mm:PinHeader_2x10_P2.54mm_Vertical, F.Cu at (143.0, 59.1)
Connections:
- A1 pad 17: unconnected-(A1-3V3-Pad17) -> +3.3V
Routing:
- net +5V: track 104.2 -> 185.1 mm
- net +3.3V: track 0.00 -> 77.5 mm, vias 0 -> 2
- net +12V: track 46.9 -> 80.0 mm
- net /D13: track 75.5 -> 76.7 mm
- net /LED: track 93.1 -> 92.4 mm
Other:
- board text added: "+12V GND"
- board text added: "+3V3 GND"
- board text added: "+5V GND"
- board text added: "A7 A6 A5 A4 A3 A2 A1 A0 AREF"
- board text added: "BREAD Slice Template: -> Conn SLC_PRTO R2 04-2025"
- board text added: "D6 D7 D8 D9 D10 D11 D12 D13"
- board text removed: "BREAD Slice Template: -> Conn SLC_TEMP R2 04-2025"
