File: hardware/BREAD_Slice_connProto.kicad_sch (KiCad schematic)
At the start: 16 parts, among them J1 Conn_01x10_Female, J2 Conn_01x08, J3 Conn_01x08

Commit message: initial commit breaking off from Slice_TEMP
Changed lines of the file:
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@@
 (kicad_sch
-	(version 20231120)
+	(version 20250114)
 	(generator "eeschema")
-	(generator_version "8.0")
+	(generator_version "9.0")
 	(paper "A4")
+	(text "Core Slice Components"
+		(exclude_from_sim no)
+		(at 16.51 17.78 0)
+		(effects
+			(font
+				(size 2.54 2.54)
+			)
+			(justify left bottom)
+		)
+	)
 	(junction
 		(at 54.61 49.53)
@@
 		)
 	)
-	(text "Core Slice Components"
-		(exclude_from_sim no)
-		(at 16.51 17.78 0)
-		(effects
-			(font
-				(size 2.54 2.54)
-			)
-			(justify left bottom)
-		)
-	)
 	(label "LED"
 		(at 40.64 68.58 180)
-		(fields_autoplaced yes)
 		(effects
 			(font
@@
 	(label "LED"
 		(at 16.51 152.4 0)
-		(fields_autoplaced yes)
 		(effects
 			(font
@@
 	(label "AREF"
 		(at 62.23 149.86 180)
-		(fields_autoplaced yes)
 		(effects
 			(font
@@
 	(label "AREF"
 		(at 73.66 160.02 0)
-		(fields_autoplaced yes)
 		(effects
 			(font
@@
 	(label "A0"
 		(at 62.23 154.94 180)
-		(fields_autoplaced yes)
 		(effects
 			(font
@@
 	(label "D13"
 		(at 73.66 135.89 0)
-		(fields_autoplaced yes)
 		(effects
 			(font
@@
 	(label "A6"
 		(at 73.66 172.72 0)
-		(fields_autoplaced yes)
 		(effects
 			(font
@@
 	(label "D7"
 		(at 16.51 157.48 0)
-		(fields_autoplaced yes)
 		(effects
 			(font
@@
 	(label "I2C_CLK"
 		(at 44.45 31.75 0)
-		(fields_autoplaced yes)
 		(effects
 			(font
@@
 	(label "RESET"
 		(at 73.66 177.8 0)
-		(fields_autoplaced yes)
 		(effects
 			(font
@@
 	(label "I2C_DAT"
 		(at 44.45 34.29 0)
-		(fields_autoplaced yes)
 		(effects
 			(font
@@
 	(label "D11"
 		(at 16.51 167.64 0)
-		(fields_autoplaced yes)
 		(effects
 			(font
@@
 	(label "A6"
 		(at 62.23 170.18 180)
-		(fields_autoplaced yes)
 		(effects
 			(font
@@
 	(label "E_STOP"
 		(at 16.51 144.78 0)
-		(fields_autoplaced yes)
 		(effects
 			(font
@@
 	(label "E_STOP"
 		(at 44.45 39.37 0)
-		(fields_autoplaced yes)
 		(effects
 			(font
@@
 	(label "D9"
 		(at 73.66 146.05 0)
-		(fields_autoplaced yes)
 		(effects
 			(font
@@
 	(label "D10"
 		(at 16.51 165.1 0)
-		(fields_autoplaced yes)
 		(effects
 			(font
@@
 	(label "A1"
 		(at 73.66 165.1 0)
-		(fields_autoplaced yes)
 		(effects
 			(font
@@
 	(label "INT"
 		(at 16.51 147.32 0)
-		(fields_autoplaced yes)
 		(effects
 			(font
@@
 	(label "A3"
 		(at 73.66 170.18 0)
-		(fields_autoplaced yes)
 		(effects
 			(font
@@
 	(label "D9"
 		(at 16.51 162.56 0)
-		(fields_autoplaced yes)
 		(effects
 			(font
@@
 	(label "D13"
 		(at 16.51 172.72 0)
-		(fields_autoplaced yes)
 		(effects
 			(font
@@
 	(label "D8"
 		(at 16.51 160.02 0)
-		(fields_autoplaced yes)
 		(effects
 			(font
@@
 	(label "SYNC"
 		(at 16.51 149.86 0)
-		(fields_autoplaced yes)
 		(effects
 			(font
@@
 	(label "D7"
 		(at 73.66 151.13 0)
-		(fields_autoplaced yes)
 		(effects
 			(font
@@
 	(label "A3"
 		(at 62.23 162.56 180)
-		(fields_autoplaced yes)
 		(effects
 			(font
@@
 	(label "RESET"
 		(at 62.23 139.7 180)
-		(fields_autoplaced yes)
 		(effects
 			(font
@@
 	(label "A1"
 		(at 62.23 157.48 180)
-		(fields_autoplaced yes)
 		(effects
 			(font
@@
 	(label "D6"
 		(at 16.51 154.94 0)
-		(fields_autoplaced yes)
 		(effects
 			(font
@@
 	(label "D10"
 		(at 73.66 143.51 0)
-		(fields_autoplaced yes)
 		(effects
 			(font
@@
 	(label "SYNC"
 		(at 44.45 44.45 0)
-		(fields_autoplaced yes)
 		(effects
 			(font
@@
 	(label "D11"
 		(at 73.66 140.97 0)
-		(fields_autoplaced yes)
 		(effects
 			(font
@@
 	(label "A2"
 		(at 73.66 167.64 0)
-		(fields_autoplaced yes)
 		(effects
 			(font
@@
 	(label "I2C_DAT"
 		(at 62.23 165.1 180)
-		(fields_autoplaced yes)
 		(effects
 			(font
@@
 	(label "D12"
 		(at 16.51 170.18 0)
-		(fields_autoplaced yes)
 		(effects
 			(font
@@
 	(label "INT"
 		(at 44.45 41.91 0)
-		(fields_autoplaced yes)
 		(effects
 			(font
@@
 	(label "A0"
 		(at 73.66 162.56 0)
-		(fields_autoplaced yes)
 		(effects
 			(font
@@
 	(label "A7"
 		(at 62.23 172.72 180)
-		(fields_autoplaced yes)
 		(effects
 			(font
@@
 	(label "I2C_CLK"
 		(at 62.23 167.64 180)
-		(fields_autoplaced yes)
 		(effects
 			(font
@@
 	(label "A2"
 		(at 62.23 160.02 180)
-		(fields_autoplaced yes)
 		(effects
 			(font
@@
 	(label "D8"
 		(at 73.66 148.59 0)
-		(fields_autoplaced yes)
 		(effects
 			(font
@@
 	(label "D6"
 		(at 73.66 153.67 0)
-		(fields_autoplaced yes)
 		(effects
 			(font
@@
 	(label "D12"
 		(at 73.66 138.43 0)
-		(fields_autoplaced yes)
 		(effects
 			(font
@@
 	(label "A7"
 		(at 73.66 175.26 0)
-		(fields_autoplaced yes)
 		(effects
 			(font
@@
 		)
 	)
+	(embedded_fonts no)
 )

Commit message: generated outputs to order
Parts:
- added J4, J5, J6, J7: Conn_02x10_Odd_Even, Connector_PinHeader_2.54mm:PinHeader_2x10_P2.54mm_Vertical, symbol Connector_Generic:Conn_02x10_Odd_Even
Connections:
- net +12V: now also J4.1 (Pin_1), J4.11 (Pin_11), J4.13 (Pin_13), J4.15 (Pin_15), J4.17 (Pin_17), J4.19 (Pin_19), J4.3 (Pin_3), J4.5 (Pin_5), J4.7 (Pin_7), J4.9 (Pin_9)
- net +5V: now also J5.1 (Pin_1), J5.11 (Pin_11), J5.13 (Pin_13), J5.15 (Pin_15), J5.17 (Pin_17), J5.19 (Pin_19), J5.3 (Pin_3), J5.5 (Pin_5), J5.7 (Pin_7), J5.9 (Pin_9), J6.1 (Pin_1), J6.11 (Pin_11), J6.13 (Pin_13), J6.15 (Pin_15), J6.17 (Pin_17), J6.19 (Pin_19), J6.3 (Pin_3), J6.5 (Pin_5), J6.7 (Pin_7), J6.9 (Pin_9)
- net GND: now also J4.10 (Pin_10), J4.12 (Pin_12), J4.14 (Pin_14), J4.16 (Pin_16), J4.18 (Pin_18), J4.2 (Pin_2), J4.20 (Pin_20), J4.4 (Pin_4), J4.6 (Pin_6), J4.8 (Pin_8), J5.10 (Pin_10), J5.12 (Pin_12), J5.14 (Pin_14), J5.16 (Pin_16), J5.18 (Pin_18), J5.2 (Pin_2), J5.20 (Pin_20), J5.4 (Pin_4), J5.6 (Pin_6), J5.8 (Pin_8), J6.10 (Pin_10), J6.12 (Pin_12), J6.14 (Pin_14), J6.16 (Pin_16), J6.18 (Pin_18), J6.2 (Pin_2), J6.20 (Pin_20), J6.4 (Pin_4), J6.6 (Pin_6), J6.8 (Pin_8), J7.10 (Pin_10), J7.12 (Pin_12), J7.14 (Pin_14), J7.16 (Pin_16), J7.18 (Pin_18), J7.2 (Pin_2), J7.20 (Pin_20), J7.4 (Pin_4), J7.6 (Pin_6), J7.8 (Pin_8)
- net +3.3V: now reaches A1.17 (3V3)
- net +3.3V: now also J7.1 (Pin_1), J7.11 (Pin_11), J7.13 (Pin_13), J7.15 (Pin_15), J7.17 (Pin_17), J7.19 (Pin_19), J7.3 (Pin_3), J7.5 (Pin_5), J7.7 (Pin_7), J7.9 (Pin_9)
- no-connect marks 6 -> 5
