File: hardware/BREAD_Slice_smtProto.kicad_pcb (KiCad board)
At the start: 2 copper layers, 70 x 100 mm, 58 parts, among them J1 Conn_01x10_Female

Commit message: generated outputs to order
Parts:
- added REF**: PinHeader_2x10_P2.54mm_Vertical, Connector_PinHeader_2.54mm:PinHeader_2x10_P2.54mm_Vertical, F.Cu at (165.9, 97.6)
- added REF**: PinHeader_2x02_P2.54mm_Vertical, Connector_PinHeader_2.54mm:PinHeader_2x02_P2.54mm_Vertical, F.Cu at (161.8, 126.7)
- moved ? 2.79 mm to (177.1, 108.3)
- moved ? 2.79 mm to (184.7, 108.3)
- moved ? 2.79 mm to (174.6, 108.3)
- moved ? 2.79 mm to (187.3, 108.3)
- moved ? 2.79 mm to (182.2, 108.3)
- moved ? 2.79 mm to (172.0, 108.3)
- moved ? 2.79 mm to (179.6, 108.3)
- moved ? 2.79 mm to (189.8, 108.3)
- moved ? 0.28 mm to (138.1, 49.2)
- moved ? 0.28 mm to (148.3, 49.2)
- moved ? 0.28 mm to (168.6, 49.2)
- moved ? 0.28 mm to (158.4, 49.2)
Connections:
- A1 pad 17: unconnected-(A1-3V3-Pad17) -> +3.3V
Routing:
- net +5V: track 104.2 -> 114.5 mm
- net GND: track 212.4 -> 222.6 mm, vias 30 -> 31
- net +3.3V: track 0.00 -> 6.97 mm
- net /LED: track 93.1 -> 92.4 mm
Other:
- board text added: "3V3 GND"
- board text added: "5V GND"
- board text added: "A0"
- board text added: "A7"
- board text added: "BREAD Slice Template: ->smtProto SLC_PRTO R2 04-2025"
- board text added: "D10"
- board text added: "D13"
- board text added: "D6"
- board text removed: "BREAD Slice Template: ->smtProto SLC_TEMP R2 04-2025"
