File: hardware/BREAD_Slice_smtProto.kicad_sch (KiCad schematic)
At the start: 14 parts, among them J1 Conn_01x10_Female

Commit message: initial commit breaking off from Slice_TEMP
Changed lines of the file:
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@@
 (kicad_sch
-	(version 20231120)
+	(version 20250114)
 	(generator "eeschema")
-	(generator_version "8.0")
+	(generator_version "9.0")
 	(paper "A4")
+	(text "Core Slice Components"
+		(exclude_from_sim no)
+		(at 16.51 17.78 0)
+		(effects
+			(font
+				(size 2.54 2.54)
+			)
+			(justify left bottom)
+		)
+	)
 	(junction
 		(at 54.61 49.53)
@@
 		)
 	)
-	(text "Core Slice Components"
-		(exclude_from_sim no)
-		(at 16.51 17.78 0)
-		(effects
-			(font
-				(size 2.54 2.54)
-			)
-			(justify left bottom)
-		)
-	)
 	(label "LED"
 		(at 40.64 68.58 180)
-		(fields_autoplaced yes)
 		(effects
 			(font
@@
 	(label "LED"
 		(at 16.51 152.4 0)
-		(fields_autoplaced yes)
 		(effects
 			(font
@@
 	(label "AREF"
 		(at 58.42 149.86 180)
-		(fields_autoplaced yes)
 		(effects
 			(font
@@
 	(label "A0"
 		(at 55.88 154.94 180)
-		(fields_autoplaced yes)
 		(effects
 			(font
@@
 	(label "D7"
 		(at 24.13 157.48 0)
-		(fields_autoplaced yes)
 		(effects
 			(font
@@
 	(label "I2C_CLK"
 		(at 44.45 31.75 0)
-		(fields_autoplaced yes)
 		(effects
 			(font
@@
 	(label "I2C_DAT"
 		(at 44.45 34.29 0)
-		(fields_autoplaced yes)
 		(effects
 			(font
@@
 	(label "D11"
 		(at 24.13 167.64 0)
-		(fields_autoplaced yes)
 		(effects
 			(font
@@
 	(label "A6"
 		(at 55.88 170.18 180)
-		(fields_autoplaced yes)
 		(effects
 			(font
@@
 	(label "E_STOP"
 		(at 16.51 144.78 0)
-		(fields_autoplaced yes)
 		(effects
 			(font
@@
 	(label "E_STOP"
 		(at 44.45 39.37 0)
-		(fields_autoplaced yes)
 		(effects
 			(font
@@
 	(label "D10"
 		(at 24.13 165.1 0)
-		(fields_autoplaced yes)
 		(effects
 			(font
@@
 	(label "INT"
 		(at 16.51 147.32 0)
-		(fields_autoplaced yes)
 		(effects
 			(font
@@
 	(label "D9"
 		(at 24.13 162.56 0)
-		(fields_autoplaced yes)
 		(effects
 			(font
@@
 	(label "D13"
 		(at 24.13 172.72 0)
-		(fields_autoplaced yes)
 		(effects
 			(font
@@
 	(label "D8"
 		(at 24.13 160.02 0)
-		(fields_autoplaced yes)
 		(effects
 			(font
@@
 	(label "SYNC"
 		(at 16.51 149.86 0)
-		(fields_autoplaced yes)
 		(effects
 			(font
@@
 	(label "A3"
 		(at 55.88 162.56 180)
-		(fields_autoplaced yes)
 		(effects
 			(font
@@
 	(label "RESET"
 		(at 59.69 139.7 180)
-		(fields_autoplaced yes)
 		(effects
 			(font
@@
 	(label "A1"
 		(at 55.88 157.48 180)
-		(fields_autoplaced yes)
 		(effects
 			(font
@@
 	(label "D6"
 		(at 24.13 154.94 0)
-		(fields_autoplaced yes)
 		(effects
 			(font
@@
 	(label "SYNC"
 		(at 44.45 44.45 0)
-		(fields_autoplaced yes)
 		(effects
 			(font
@@
 	(label "I2C_DAT"
 		(at 63.5 165.1 180)
-		(fields_autoplaced yes)
 		(effects
 			(font
@@
 	(label "D12"
 		(at 24.13 170.18 0)
-		(fields_autoplaced yes)
 		(effects
 			(font
@@
 	(label "INT"
 		(at 44.45 41.91 0)
-		(fields_autoplaced yes)
 		(effects
 			(font
@@
 	(label "A7"
 		(at 55.88 172.72 180)
-		(fields_autoplaced yes)
 		(effects
 			(font
@@
 	(label "I2C_CLK"
 		(at 63.5 167.64 180)
-		(fields_autoplaced yes)
 		(effects
 			(font
@@
 	(label "A2"
 		(at 55.88 160.02 180)
-		(fields_autoplaced yes)
 		(effects
 			(font
@@
 		)
 	)
+	(embedded_fonts no)
 )

Commit message: generated outputs to order
Connections:
- net +3.3V: now reaches A1.17 (3V3)
- no-connect marks 6 -> 5
Changed lines of the file:
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@@
-	)
-	(no_connect
-		(at 43.18 129.54)
 	)
 	(no_connect
@@
 					(unit 1)
 				)
+			)
+		)
+	)
+	(symbol
+		(lib_id "power:+3.3V")
+		(at 43.18 129.54 0)
+		(unit 1)
+		(exclude_from_sim no)
+		(in_bom yes)
+		(on_board yes)
+		(dnp no)
+		(property "Reference" "#PWR014"
+			(at 43.18 133.35 0)
+			(effects
+				(font
+					(size 1.27 1.27)
+				)
+				(hide yes)
+			)
+		)
+		(property "Value" "+3.3V"
+			(at 41.402 125.73 0)
+			(effects
+				(font
+					(size 1.27 1.27)
+				)
+			)
+		)
+		(property "Footprint" ""
+			(at 43.18 129.54 0)
+			(effects
+				(font
+					(size 1.27 1.27)
+				)
+				(hide yes)
+			)
+		)
+		(property "Datasheet" ""
+			(at 43.18 129.54 0)
+			(effects
+				(font
+					(size 1.27 1.27)
+				)
+				(hide yes)
+			)
+		)
+		(property "Description" "Power symbol creates a global label with name \"+3.3V\""
+			(at 43.18 129.54 0)
+			(effects
+				(font
+					(size 1.27 1.27)
+				)
+				(hide yes)
+			)
+		)
+		(pin "1"
+		)
+		(instances
+			(project ""
+				(path "/66043bca-a260-4915-9fce-8a51d324c687"
+					(reference "#PWR014")
+					(unit 1)
+				)
