File: hardware/BREAD_Slice_thProto.kicad_pcb (KiCad board)
At the start: 2 copper layers, 70 x 100 mm, 31 parts, among them J1 Conn_01x10_Female

Commit message: generated outputs to order
Routing:
- net /LED: track 93.1 -> 92.1 mm
- net +5V: track 109.7 -> 108.7 mm
Other:
- board text added: "BREAD Slice Template: -> thProto SLC_PRTO R2 04-2025"
- board text removed: "BREAD Slice Template: -> thProto SLC_TEMP R2 04-2025"
Changed lines of the file:
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@@
 		(grid_origin 122.6 139.8)
 		(pcbplotparams
-			(layerselection 0x00000000_00000000_55555555_5755f5ff)
+			(layerselection 0x00000000_00000000_55555555_575555ff)
 			(plot_on_all_layers_selection 0x00000000_00000000_00000000_00000000)
 			(disableapertmacros no)
@@
 			(sketchdnponfab yes)
 			(crossoutdnponfab yes)
-			(subtractmaskfromsilk no)
+			(subtractmaskfromsilk yes)
 			(outputformat 1)
 			(mirror no)
 			(drillshape 0)
 			(scaleselection 1)
-			(outputdirectory "Gerbers/")
+			(outputdirectory "outputs-tht")
 		)
 	)
@@
 	(gr_line
 		(start 127.600001 129.149999)
-		(end 124.6 129.149999)
+		(end 124.3 129.149999)
 		(stroke
 			(width 0.1)
@@
 	)
 	(gr_line
-		(start 124.6 129.149999)
-		(end 124.6 107.1)
+		(start 124.3 129.149999)
+		(end 124.3 107.1)
 		(stroke
 			(width 0.1)
@@
 	)
 	(gr_line
-		(start 124.6 107.1)
+		(start 124.3 107.1)
 		(end 115.3 107.1)
 		(stroke
@@
 		)
 	)
-	(gr_text "BREAD Slice\nTemplate:\n-> thProto\nSLC_TEMP\nR2 04-2025"
-		(at 128 103.5 270)
+	(gr_text "BREAD Slice\nTemplate:\n-> thProto\nSLC_PRTO\nR2 04-2025"
+		(at 128.4 103.5 270)
 		(layer "F.SilkS")
 		(effects
@@
 		(at 129.85 120.955)
 		(size 0.5)
-		(drill 0.2)
+		(drill 0.3)
 		(layers "F.Cu" "B.Cu")
 		(free yes)
@@
 		(at 131.15 120.255)
 		(size 0.5)
-		(drill 0.2)
+		(drill 0.3)
 		(layers "F.Cu" "B.Cu")
 		(free yes)
@@
 		(at 131.15 118.755)
 		(size 0.5)
-		(drill 0.2)
+		(drill 0.3)
 		(layers "F.Cu" "B.Cu")
 		(free yes)
@@
 		(at 130.05 117.955)
 		(size 0.5)
-		(drill 0.2)
+		(drill 0.3)
 		(layers "F.Cu" "B.Cu")
 		(free yes)
@@
 		(at 132.35 117.955)
 		(size 0.5)
-		(drill 0.2)
+		(drill 0.3)
 		(layers "F.Cu" "B.Cu")
 		(free yes)
@@
 		(at 130.75 120.955)
 		(size 0.5)
-		(drill 0.2)
+		(drill 0.3)
 		(layers "F.Cu" "B.Cu")
 		(free yes)
@@
 	)
 	(segment
-		(start 168.675 133.375)
-		(end 168.675 110.025)
+		(start 165.05 137)
+		(end 168.25 133.8)
 		(width 1.5)
 		(layer "F.Cu")
@@
 	)
 	(segment
-		(start 163.71 105.06)
-		(end 157.85 105.06)
+		(start 168.675 133.375)
+		(end 168.675 110.025)
 		(width 1.5)
 		(layer "F.Cu")
@@
 	)
 	(segment
-		(start 166.325 107.875)
-		(end 166.325 112.955)
+		(start 163.71 105.06)
+		(end 157.85 105.06)
 		(width 1.5)
 		(layer "F.Cu")
@@
 	)
 	(segment
-		(start 135.25 133.25)
-		(end 139.85 137.85)
+		(start 135.25 129.2)
+		(end 135.25 132.75)
 		(width 1.5)
 		(layer "F.Cu")
@@
 	)
 	(segment
-		(start 135.25 129.2)
-		(end 135.25 133.25)
+		(start 166.325 107.875)
+		(end 166.325 112.955)
 		(width 1.5)
 		(layer "F.Cu")
@@
 	)
 	(segment
-		(start 164.2 137.85)
-		(end 168.25 133.8)
+		(start 135.25 132.75)
+		(end 139.5 137)
 		(width 1.5)
 		(layer "F.Cu")
@@
 	)
 	(segment
-		(start 139.85 137.85)
-		(end 164.2 137.85)
+		(start 139.5 137)
+		(end 165.05 137)
 		(width 1.5)
 		(layer "F.Cu")
@@
 	)
 	(segment
-		(start 124.925 127.125)
-		(end 124.925 115.825)
+		(start 139.3 138.5)
+		(end 134 133.2)
 		(width 0.5)
 		(layer "F.Cu")
@@
 	)
 	(segment
-		(start 126.45 128.65)
-		(end 124.925 127.125)
+		(start 125.8 114.95)
+		(end 142.34 114.95)
 		(width 0.5)
 		(layer "F.Cu")
@@
 	)
 	(segment
-		(start 177 138.35)
-		(end 176.3 139.05)
+		(start 142.34 114.95)
+		(end 142.61 115.22)
 		(width 0.5)
 		(layer "F.Cu")
@@
 	)
 	(segment
-		(start 176.3 139.05)
-		(end 139.352944 139.05)
+		(start 177.1 135.555769)
+		(end 177.1 138)
 		(width 0.5)
 		(layer "F.Cu")
@@
 	)
 	(segment
-		(start 177 135.455769)
-		(end 175.677 134.132769)
+		(start 134 133.2)
+		(end 134 131.1)
 		(width 0.5)
 		(layer "F.Cu")
@@
 	)
 	(segment
-		(start 133.7 130.8)
-		(end 131.55 128.65)
+		(start 126.1 128.3)
+		(end 125.2 127.4)
 		(width 0.5)
 		(layer "F.Cu")
@@
 	)
 	(segment
-		(start 177 135.455769)
-		(end 177 138.35)
+		(start 125.2 127.4)
+		(end 125.2 115.55)
 		(width 0.5)
 		(layer "F.Cu")
@@
 	)
 	(segment
-		(start 125.8 114.95)
-		(end 142.34 114.95)
+		(start 177.1 138)
+		(end 176.6 138.5)
 		(width 0.5)
 		(layer "F.Cu")
@@
 	)
 	(segment
-		(start 131.55 128.65)
-		(end 126.45 128.65)
+		(start 131.2 128.3)
+		(end 126.1 128.3)
 		(width 0.5)
 		(layer "F.Cu")
@@
 	)
 	(segment
-		(start 142.34 114.95)
-		(end 142.61 115.22)
+		(start 125.2 115.55)
+		(end 125.8 114.95)
 		(width 0.5)
 		(layer "F.Cu")
@@
 	)
 	(segment
-		(start 133.7 133.397056)
-		(end 133.7 130.8)
+		(start 176.6 138.5)
+		(end 139.3 138.5)
 		(width 0.5)
 		(layer "F.Cu")
@@
 	)
 	(segment
-		(start 124.925 115.825)
-		(end 125.8 114.95)
+		(start 175.677 134.132769)
+		(end 177.1 135.555769)
 		(width 0.5)
 		(layer "F.Cu")
@@
 	)
 	(segment
-		(start 139.352944 139.05)
-		(end 133.7 133.397056)
+		(start 134 131.1)
+		(end 131.2 128.3)
 		(width 0.5)
 		(layer "F.Cu")
