File: hardware/BREAD_Slice.kicad_pcb (KiCad board)
At the start: 2 copper layers, 70 x 100 mm, 31 parts, among them J1 Conn_01x10_Female

Commit message: clear erc and drc but this board needs some rebuild help long term
Parts:
- removed the REF** at (161.5, 94.7)
- removed the REF** at (161.6, 107.8)
- removed the REF** at (151.4, 91.1)
- removed the REF** at (166.3, 107.9)
- added J2: Conn_01x03_Pin, Connector_PinHeader_2.54mm:PinHeader_1x03_P2.54mm_Vertical, F.Cu at (166.3, 107.9)
- added J3: Conn_01x02_Pin, Connector_PinHeader_2.54mm:PinHeader_1x02_P2.54mm_Vertical, F.Cu at (166.4, 97.2)
- added J4: Conn_01x02_Pin, Connector_PinHeader_2.54mm:PinHeader_1x02_P2.54mm_Vertical, F.Cu at (161.6, 124.8)
- added J5: Conn_01x05_Pin, Connector_PinHeader_2.54mm:PinHeader_1x05_P2.54mm_Vertical, F.Cu at (151.4, 91.1)
- added J6: Conn_01x06_Pin, Connector_PinHeader_2.54mm:PinHeader_1x06_P2.54mm_Vertical, F.Cu at (161.6, 107.8)
- added J7: Conn_01x03_Pin, Connector_PinHeader_2.54mm:PinHeader_1x03_P2.54mm_Vertical, F.Cu at (161.5, 94.7)
- added J8: Conn_01x03_Pin, Connector_PinHeader_2.54mm:PinHeader_1x03_P2.54mm_Vertical, F.Cu at (166.3, 116.5)
- J1: value Conn_01x10_Female -> Conn_01x10_Socket
- renumbered H3 to H2, H2 to H3
Routing:
- net /RESET: track 0.00 -> 12.3 mm
- net GND: track 364.3 -> 371.0 mm, vias 14 -> 15
- net /AREF: track 0.00 -> 6.47 mm
- net /I2C_DAT: track 46.0 -> 50.5 mm
- net /I2C_CLK: track 46.3 -> 49.6 mm
Other:
- board text added: "AREF"
- board text added: "RESET"
