File: hardware/BREAD_Slice.kicad_pcb (KiCad board)
At the start: 2 copper layers, 70 x 100 mm, 34 parts, among them J1 Conn_01x10_Socket, J2 Conn_01x03_Pin, J3 Conn_01x02_Pin, J4 Conn_01x02_Pin, J5 Conn_01x05_Pin, J6 Conn_01x06_Pin, J7 Conn_01x03_Pin, J8 Conn_01x03_Pin

Commit message: review and revise board and update footprints
Parts:
- removed the ? at (158.9, 84.3)
- removed the ? at (156.4, 84.3)
- removed the ? at (153.8, 84.3)
- removed the ? at (161.4, 84.3)
- removed the ? at (151.3, 84.3)
- added REF**: 0805_HandSolder_TH_AnnularPad, KMLib_Proto:0805_HandSolder_TH_AnnularPad, F.Cu at (153.2, 81.6)
- added REF**: 0805_HandSolder_TH_AnnularPad, KMLib_Proto:0805_HandSolder_TH_AnnularPad, F.Cu at (153.2, 86.5)
- added REF**: 0805_HandSolder_TH_AnnularPad, KMLib_Proto:0805_HandSolder_TH_AnnularPad, F.Cu at (163.4, 86.5)
- added REF**: 0805_HandSolder_TH_AnnularPad, KMLib_Proto:0805_HandSolder_TH_AnnularPad, F.Cu at (163.4, 84.1)
- added REF**: 0805_HandSolder_TH_AnnularPad, KMLib_Proto:0805_HandSolder_TH_AnnularPad, F.Cu at (163.4, 81.6)
- added REF**: 0805_HandSolder_TH_AnnularPad, KMLib_Proto:0805_HandSolder_TH_AnnularPad, F.Cu at (153.2, 84.1)
- added Ref**: Val**, KMLib_Proto:1206_HandSolder_Dual_TH_AnnularPad, F.Cu at (143.9, 59.6)
- added Ref**: Val**, KMLib_Proto:1206_HandSolder_Dual_TH_AnnularPad, F.Cu at (164.2, 59.6)
- ? (x2): footprint kicad_wrk:PROTO-SOT-23-6 -> KMLib_Proto:SOT-23-6_TH_AnnularPad
- D1: footprint SparkFun-LED:WS2812-5050-4PIN -> KMLib_IC_SMD:WS2812-5050-4PIN
- HS1: footprint KML-Custom:Thermal Pad -> KMLib_Mounting:Thermal Pad
- REF**: value protogrid_5x20 -> Grid_TH_AnnularPad_5x20_2.54mm; footprint proto:protogrid_5x20 -> KMLib_Proto:Grid_TH_AnnularPad_5x20_2.54mm
- REF** (x2): value protogrid_5x15 -> Grid_TH_AnnularPad_5x15_2.54mm; footprint proto:protogrid_5x15 -> KMLib_Proto:Grid_TH_AnnularPad_5x15_2.54mm
Connections:
- REF** pad 10: GND -> (no net)
- REF** pad 12: GND -> (no net)
- REF** pad 14: GND -> (no net)
- REF** pad 16: GND -> (no net)
- REF** pad 18: GND -> (no net)
- REF** pad 2: GND -> (no net)
- REF** pad 20: GND -> (no net)
- REF** pad 22: GND -> (no net)
- REF** pad 24: GND -> (no net)
- REF** pad 26: GND -> (no net)
- REF** pad 28: GND -> (no net)
- REF** pad 30: GND -> (no net)
- REF** pad 32: GND -> (no net)
- REF** pad 34: GND -> (no net)
- REF** pad 36: GND -> (no net)
- REF** pad 4: GND -> (no net)
- REF** pad 6: GND -> (no net)
- REF** pad 8: GND -> (no net)
- REF** pad 1: GND -> (no net)
- REF** pad 11: GND -> (no net)
- REF** pad 13: GND -> (no net)
- REF** pad 15: GND -> (no net)
- REF** pad 17: GND -> (no net)
- REF** pad 19: GND -> (no net)
- REF** pad 21: GND -> (no net)
- REF** pad 23: GND -> (no net)
- REF** pad 25: GND -> (no net)
- REF** pad 27: GND -> (no net)
- REF** pad 29: GND -> (no net)
- REF** pad 3: GND -> (no net)
- REF** pad 31: GND -> (no net)
- REF** pad 33: GND -> (no net)
- REF** pad 35: GND -> (no net)
- REF** pad 5: GND -> (no net)
- REF** pad 7: GND -> (no net)
- REF** pad 9: GND -> (no net)
