File: hardware/BREAD_Slice.kicad_sch (KiCad schematic)
At the start: 21 parts, among them J1 Conn_01x10_Socket, J2 Conn_01x03_Pin, J3 Conn_01x02_Pin, J4 Conn_01x02_Pin, J5 Conn_01x05_Pin, J6 Conn_01x06_Pin, J7 Conn_01x03_Pin, J8 Conn_01x03_Pin

Commit message: review and revise board and update footprints
Parts:
- D1: footprint SparkFun-LED:WS2812-5050-4PIN -> KMLib_IC_SMD:WS2812-5050-4PIN
- HS1: footprint KML-Custom:Thermal Pad -> KMLib_Mounting:Thermal Pad
Changed lines of the file:
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@@
 			)
 		)
-		(property "Footprint" "KML-Custom:Thermal Pad"
+		(property "Footprint" "KMLib_Mounting:Thermal Pad"
 			(at 82.55 112.0648 0)
 			(effects
@@
 			)
 		)
-		(property "Footprint" "SparkFun-LED:WS2812-5050-4PIN"
+		(property "Footprint" "KMLib_IC_SMD:WS2812-5050-4PIN"
 			(at 86.36 76.2 0)
 			(effects
